File: Anachron/Peripherals.kicad_sch (KiCad schematic)
At the start: 21 parts, among them J3 Motor Pads, SW2 Pad, U4 BMI270, U5 MAX98357A

Commit message: routing done?
Parts:
- renumbered J3 to MP1
Connections:
- net +3.3V: now also U5.8 (VDD)
- net EN_A: no longer S6.B
- net GND: now also U5.11 (GND), U5.15 (GND)
- net EN_B: now reaches C20.1, R17.2
- net EN_B: now also S6.B
Changed lines of the file:
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@@
 	)
 	(junction
-		(at 66.04 165.1)
-		(diameter 0)
-		(color 0 0 0 0)
-	)
-	(junction
 		(at 247.65 129.54)
 		(diameter 0)
@@
 	)
 	(junction
+		(at 44.45 165.1)
+		(diameter 0)
+		(color 0 0 0 0)
+	)
+	(junction
 		(at 97.79 105.41)
 		(diameter 0)
@@
 	)
 	(junction
+		(at 66.04 165.1)
+		(diameter 0)
+		(color 0 0 0 0)
+	)
+	(junction
 		(at 194.31 76.2)
 		(diameter 0)
@@
 		(color 0 0 0 0)
 	)
-	(junction
-		(at 48.26 165.1)
-		(diameter 0)
-		(color 0 0 0 0)
-	)
 	(no_connect
 		(at 198.12 66.04)
@@
 	(wire
 		(pts
-			(xy 64.77 158.75) (xy 66.04 158.75)
+			(xy 44.45 165.1) (xy 44.45 166.37)
 		)
 		(stroke
@@
 	(wire
 		(pts
-			(xy 45.72 88.9) (xy 45.72 104.14)
+			(xy 64.77 158.75) (xy 66.04 158.75)
 		)
 		(stroke
@@
 	(wire
 		(pts
-			(xy 194.31 125.73) (xy 207.01 125.73)
+			(xy 45.72 88.9) (xy 45.72 104.14)
 		)
 		(stroke
@@
 	(wire
 		(pts
-			(xy 250.19 59.69) (xy 250.19 66.04)
+			(xy 194.31 125.73) (xy 207.01 125.73)
 		)
 		(stroke
@@
 	(wire
 		(pts
-			(xy 57.15 162.56) (xy 57.15 172.72)
+			(xy 250.19 59.69) (xy 250.19 66.04)
 		)
 		(stroke
@@
 	(wire
 		(pts
-			(xy 250.19 66.04) (xy 250.19 76.2)
+			(xy 57.15 162.56) (xy 57.15 172.72)
 		)
 		(stroke
@@
 	(wire
 		(pts
-			(xy 223.52 142.24) (xy 233.68 142.24)
+			(xy 250.19 66.04) (xy 250.19 76.2)
 		)
 		(stroke
@@
 	(wire
 		(pts
-			(xy 64.77 163.83) (xy 66.04 163.83)
+			(xy 223.52 142.24) (xy 233.68 142.24)
 		)
 		(stroke
@@
 	(wire
 		(pts
+			(xy 64.77 163.83) (xy 66.04 163.83)
+		)
+		(stroke
+			(width 0)
+			(type default)
+		)
+	)
+	(wire
+		(pts
 			(xy 186.69 59.69) (xy 186.69 60.96)
 		)
@@
 	(wire
 		(pts
-			(xy 48.26 165.1) (xy 48.26 166.37)
+			(xy 48.26 160.02) (xy 48.26 166.37)
 		)
 		(stroke
@@
 	(wire
 		(pts
+			(xy 66.04 163.83) (xy 66.04 165.1)
+		)
+		(stroke
+			(width 0)
+			(type default)
+		)
+	)
+	(wire
+		(pts
 			(xy 194.31 76.2) (xy 198.12 76.2)
 		)
@@
 	(wire
 		(pts
-			(xy 66.04 163.83) (xy 66.04 165.1)
+			(xy 97.79 90.17) (xy 97.79 105.41)
 		)
 		(stroke
@@
 	(wire
 		(pts
-			(xy 97.79 90.17) (xy 97.79 105.41)
+			(xy 48.26 104.14) (xy 45.72 104.14)
 		)
 		(stroke
@@
 	(wire
 		(pts
-			(xy 48.26 104.14) (xy 45.72 104.14)
+			(xy 73.66 119.38) (xy 73.66 120.65)
 		)
 		(stroke
@@
 	(wire
 		(pts
-			(xy 73.66 119.38) (xy 73.66 120.65)
+			(xy 44.45 165.1) (xy 66.04 165.1)
 		)
 		(stroke
@@
 	(wire
 		(pts
-			(xy 48.26 160.02) (xy 48.26 165.1)
-		)
-		(stroke
-			(width 0)
-			(type default)
-		)
-	)
-	(wire
-		(pts
 			(xy 199.39 142.24) (xy 213.36 142.24)
 		)
@@
 	(wire
 		(pts
-			(xy 44.45 158.75) (xy 44.45 166.37)
+			(xy 44.45 158.75) (xy 44.45 165.1)
 		)
 		(stroke
@@
 		)
 	)
-	(wire
-		(pts
-			(xy 48.26 165.1) (xy 66.04 165.1)
-		)
-		(stroke
-			(width 0)
-			(type default)
-		)
-	)
 	(label "Gain_Control"
 		(at 199.39 142.24 0)
@@
 		(dnp no)
 		(fields_autoplaced yes)
-		(property "Reference" "J3"
+		(property "Reference" "MP1"
 			(at 219.71 101.5999 0)
 			(show_name no)
@@
 			(project "Anachron"
 				(path "/05e7c6ef-b370-43a4-82c0-82f37f32c760/b0f66910-b91e-42a0-b088-9df41a9888a7"
-					(reference "J3")
+					(reference "MP1")
 					(unit 1)
 				)

Commit message: more changes!
Other:
- note added: "Buttons (ADC Ladder)"
- note added: "I2S Amplifier (MAX98357A)"
- note added: "IMU (BMI270)"
- note added: "Rotary Encoder (EC05)"
- moved on the sheet: C13, C14, C15, C16, C17, C20, C21, MP1, R13, R14, R15, R16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
