File: Anachron/Anachron.kicad_sch (KiCad schematic)
At the start: 19 parts, among them J1 USB4520-03-0-A, Q1 AO3401A, SW1 Pad, U1 AP2112K-3.3TRG1, U2 MCP73831T-2ACI_OT

Commit message: pcb placement starting
Parts:
- BT1: footprint (none) -> Connector_JST:JST_PH_B2B-PH-K_1x02_P2.00mm_Vertical
- C1, C2, C3, C4, C5, R1, R2, R3, R4, R5: footprint (none) -> Capacitor_SMD:C_0603_1608Metric
- D1: footprint SOT23-6L_STM -> footprints:SOT23-6L_STM
- D3: footprint (none) -> footprints:CR_5817PL-TP_MCC
- J1: footprint USB4520-03-0-A_REVA:GCT_USB4520-03-0-A_REVA -> footprints:GCT_USB4520-03-0-A_REVA
- U1: footprint SOT_RG1_DIO -> footprints:SOT_RG1_DIO
- U2: footprint SOT95P270X145-5N -> footprints:SOT95P270X145-5N
Connections:
- net GND: no longer D1.5
- net VBUS: now also D1.5
- net VSYS: now also SW1.2 (B); no longer SW1.1 (A)
- net EN Mode: now reaches U1.3 (EN)
- net EN Mode: now also SW1.1 (A); no longer SW1.2 (B)
Other:
- moved on the sheet: BT1, C1, C2, C3, D2, D3, Q1, R3, R4, R5, SW1, U2

Commit message: mcu and screen page
Parts:
- removed BT1: Battery_Cell, Connector_JST:JST_PH_B2B-PH-K_1x02_P2.00mm_Vertical, symbol Device:Battery_Cell
- removed C1: 100nF, Capacitor_SMD:C_0603_1608Metric, symbol Device:C_Small
- removed C2, C3: 4.7uF, Capacitor_SMD:C_0603_1608Metric, symbol Device:C_Small
- removed C4, C5: 1uF, Capacitor_SMD:C_0603_1608Metric, symbol Device:C_Small
- removed D1: USBLC6-2SC6, footprints:SOT23-6L_STM, symbol symbols:USBLC6-2SC6
- removed D2: LED_Small, symbol Device:LED_Small
- removed D3: SM5817PL-TP, footprints:CR_5817PL-TP_MCC, symbol Device:D_Small
- removed J1: USB4520-03-0-A, footprints:GCT_USB4520-03-0-A_REVA, symbol symbols:USB4520-03-0-A_REVA
- removed Q1: AO3401A, Package_TO_SOT_SMD:SOT-23, symbol Transistor_FET:AO3401A
- removed R1, R2: 5k1, Capacitor_SMD:C_0603_1608Metric, symbol Device:R_Small_US
- removed R3: 4k7, Capacitor_SMD:C_0603_1608Metric, symbol Device:R_Small_US
- removed R4: 470, Capacitor_SMD:C_0603_1608Metric, symbol Device:R_Small_US
- removed R5: 10k, Capacitor_SMD:C_0603_1608Metric, symbol Device:R_Small_US
- removed SW1: Pad, Jumper:SolderJumper-2_P1.3mm_Open_RoundedPad1.0x1.5mm, symbol Switch:SW_SPST
- removed U1: AP2112K-3.3TRG1, footprints:SOT_RG1_DIO, symbol symbols:AP2112K-3.3TRG1
- removed U2: MCP73831T-2ACI_OT, footprints:SOT95P270X145-5N, symbol symbols:MCP73831T-2ACI_OT
Connections:
- no-connect marks 3 -> 0
Other:
- added sheet MCU + Screen (MCUScreen.kicad_sch)
- added sheet Power (power.kicad_sch)
- note removed: "Charging Current: I = 1000/R3 I = 1000/4.7 = 212 mA"
- note removed: "FOOTPRINT FOR BATTERY AND LED"

Commit message: layout power
Other:
- added sheet Peripherals (Peripherals.kicad_sch)
Changed lines of the file:
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@@
+	)
+	(sheet
+		(at 110.49 58.42)
+		(size 25.4 11.43)
+		(exclude_from_sim no)
+		(in_bom yes)
+		(on_board yes)
+		(dnp no)
+		(fields_autoplaced yes)
+		(stroke
+			(width 0.1524)
+			(type solid)
+		)
+		(fill
+			(color 0 0 0 0)
+		)
+		(property "Sheetname" "Peripherals"
+			(at 110.49 57.7084 0)
+			(show_name no)
+			(do_not_autoplace no)
+			(effects
+				(font
+					(size 1.27 1.27)
+				)
+				(justify left bottom)
+			)
+		)
+		(property "Sheetfile" "Peripherals.kicad_sch"
+			(at 110.49 70.4346 0)
+			(show_name no)
+			(do_not_autoplace no)
+			(effects
+				(font
+					(size 1.27 1.27)
+				)
+				(justify left top)
+			)
+		)
+		(instances
+			(project "Anachron"
+				(path "/05e7c6ef-b370-43a4-82c0-82f37f32c760"
+					(page "3")
+				)
+			)
+		)
 	)
 	(sheet

Commit message: layed everything outttt
Other:
- sheet MCU + Screen ports: added ADC_Button, AMP_BCLK, AMP_DIN, AMP_LRCLK, AMP_Mode, EN_A, EN_B, IMU_INT1, IMU_INT2, MCU_D_N, MCU_D_P, SCL, SDA; removed none
- sheet Peripherals ports: added ADC_Button, AMP_BCLK, AMP_DIN, AMP_LRCLK, AMP_Mode, EN_A, EN_B, IMU_INT1, IMU_INT2, SCL, SDA; removed none
- sheet Power ports: added MCU_D_N, MCU_D_P; removed none

Commit message: layout power
Other:
- sheet MCU + Screen ports: added none; removed ADC_Button, AMP_BCLK, AMP_DIN, AMP_LRCLK, AMP_Mode, EN_A, EN_B, IMU_INT1, IMU_INT2, MCU_D_N, MCU_D_P, SCL, SDA
- sheet Peripherals ports: added none; removed ADC_Button, AMP_BCLK, AMP_DIN, AMP_LRCLK, AMP_Mode, EN_A, EN_B, IMU_INT1, IMU_INT2, SCL, SDA
- sheet Power ports: added none; removed MCU_D_N, MCU_D_P
