File: Anachron/MCUScreen.kicad_sch (KiCad schematic)
At the start: 24 parts, among them J2 FFC2B35-18-G_REVA2, U3 ESP32-S3 N8R8, Y1 32.768kHz

Commit message: layout power
Parts:
- removed R19, R20: 10k, Resistor_SMD:R_0603_1608Metric, symbol Device:R_Small_US
- removed TP4: TX, TestPoint:TestPoint_Pad_D1.5mm, symbol Connector:TestPoint
- removed TP5: RX, TestPoint:TestPoint_Pad_D1.5mm, symbol Connector:TestPoint
- removed TP6: SDA, TestPoint:TestPoint_Pad_D1.5mm, symbol Connector:TestPoint
- removed TP7: SCL, TestPoint:TestPoint_Pad_D1.5mm, symbol Connector:TestPoint
- J2: footprint FFC2B35-18-G_REVA2:GCT_FFC2B35-18-G_REVA2 -> footprints:GCT_FFC2B35-18-G_REVA2
- S1, S2: footprint TS18-5-25-SL-160-SMT-TR:SW_TS18-5-25-SL-160-SMT-TR -> footprints:SW_TS18-5-25-SL-160-SMT-TR
Connections:
- net LCD_BL: no longer U3.4 (IO4)
- net LCD_CS: no longer U3.18 (IO10)
- net LCD_IO0: no longer U3.19 (IO11)
- net LCD_IO1: no longer U3.21 (IO13)
- net LCD_IO2: no longer U3.22 (IO14)
- net LCD_IO3: no longer U3.17 (IO9)
- net LCD_RST: no longer U3.24 (IO47)
- net LCD_SCLK: no longer U3.20 (IO12)
- net LCD_TE: no longer U3.23 (IO21)
- net SCL: no longer U3.39 (IO1)
- net SDA: no longer U3.38 (IO2)
- net TP_INT: no longer U3.5 (IO5)
- net TP_RST: no longer U3.25 (IO48)
- net ADC_Bat renamed Battery ADC
- net Battery ADC: no longer U3.7 (IO7)
- net ADC_Button: no longer names the net of U3.6 (IO6)
- net AMP_BCLK: no longer names the net of U3.33 (IO40)
- net AMP_DIN: no longer names the net of U3.35 (IO42)
- net AMP_LRCLK: no longer names the net of U3.34 (IO41)
- net AMP_Mode: no longer names the net of U3.12 (IO8)
- net EN_A: no longer names the net of U3.31 (IO38)
- net EN_B: no longer names the net of U3.32 (IO39)
- net IMU_INT1: no longer names the net of U3.10 (IO17)
- net IMU_INT2: no longer names the net of U3.11 (IO18)
Other:
- moved on the sheet: C10, C11, C12, C6, C7, C8, C9, J2, R11, R12, R6, R7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
