File: Anachron/MCUScreen.kicad_sch (KiCad schematic)
At the start: 17 parts, among them J2 FFC2B35-18-G_REVA2, U3 ESP32-S3 N8R8, Y1 32.768kHz

Commit message: layout power
Parts:
- C11, C12: value 15pF -> 4pF
Connections:
- net OSC_N: now reaches C11.1, R9.1, Y1.1
- net OSC_P: now reaches C12.1, R10.2, Y1.2
- net XTAL_32K_N renamed MCU_OSC_N
- net XTAL_32K_P renamed MCU_OSC_P
Other:
- note added: "C = 2 x (C_Load - C_Stray) C = 2 x (7pF - 5pF) C = 2 x 2pF C = 4pF"
- note removed: "C = 2 x (C_Load - C_Stray) C = 2 x (12.5pF - 5pF) C = 2 x 7.5pF C = 15pF"
- note removed: "FIND A OSC PART MAKE SURE LOAD IS 12.5pF OR CHANGE THE C VALUES"
- moved on the sheet: C11, C12, R10, R9, Y1

Commit message: layout power
Parts:
- removed R10: 0, Capacitor_SMD:C_0603_1608Metric, symbol Device:R_Small_US
- added R11, R12: 100k, Resistor_SMD:R_0603_1608Metric, symbol Device:R_Small_US
- C10, C11, C12, C9: footprint Capacitor_SMD:C_0805_2012Metric -> Capacitor_SMD:C_0603_1608Metric
- R6, R7, R8, R9: footprint Capacitor_SMD:C_0603_1608Metric -> Resistor_SMD:R_0603_1608Metric
- S1, S2: footprint TS18-5-25-SL-160-SMT-TR:SW_TS18-5-25-SL-160-SMT-TR -> footprints:SW_TS18-5-25-SL-160-SMT-TR
Connections:
- net OSC_P is gone; now on net MCU_OSC_P: C12.1, Y1.2
- net BOOT: no longer C10.1
- net GND: now also R12.2
- net TP_SCL renamed SCL
- net TP_SDA renamed SDA
- new net Battery ADC: C10.1, R11.2, R12.1
- new net VBAT: R11.1

Commit message: layed everything outttt
Parts:
- added R19, R20: 10k, Resistor_SMD:R_0603_1608Metric, symbol Device:R_Small_US
- added TP4: TX, TestPoint:TestPoint_Pad_D1.5mm, symbol Connector:TestPoint
- added TP5: RX, TestPoint:TestPoint_Pad_D1.5mm, symbol Connector:TestPoint
- added TP6: SDA, TestPoint:TestPoint_Pad_D1.5mm, symbol Connector:TestPoint
- added TP7: SCL, TestPoint:TestPoint_Pad_D1.5mm, symbol Connector:TestPoint
- J2: footprint footprints:GCT_FFC2B35-18-G_REVA2 -> FFC2B35-18-G_REVA2:GCT_FFC2B35-18-G_REVA2
- S1, S2: footprint footprints:SW_TS18-5-25-SL-160-SMT-TR -> TS18-5-25-SL-160-SMT-TR:SW_TS18-5-25-SL-160-SMT-TR
Connections:
- net Battery ADC is gone; now on net ADC_Bat: C10.1, R11.2, R12.1
- net +3.3V: now also R19.2, R20.2
- net LCD_BL: now also U3.4 (IO4)
- net LCD_CS: now also U3.18 (IO10)
- net LCD_IO0: now also U3.19 (IO11)
- net LCD_IO1: now also U3.21 (IO13)
- net LCD_IO2: now also U3.22 (IO14)
- net LCD_IO3: now also U3.17 (IO9)
- net LCD_RST: now also U3.24 (IO47)
- net LCD_SCLK: now also U3.20 (IO12)
- net LCD_TE: now also U3.23 (IO21)
- net MCU_RX: now also TP4.1
- net MCU_TX: now also TP5.1
- net SCL: now also U3.39 (IO1), R19.1, TP7.1
- net SDA: now also U3.38 (IO2), R20.1, TP6.1
- net TP_INT: now also U3.5 (IO5)
- net TP_RST: now also U3.25 (IO48)
- net IMU_INT1: now reaches U3.10 (IO17)
- net IMU_INT2: now reaches U3.11 (IO18)
- net AMP_Mode: now reaches U3.12 (IO8)
- net EN_A: now reaches U3.31 (IO38)
- net EN_B: now reaches U3.32 (IO39)
- net AMP_BCLK: now reaches U3.33 (IO40)
- net AMP_LRCLK: now reaches U3.34 (IO41)
- net AMP_DIN: now reaches U3.35 (IO42)
- net ADC_Button: now reaches U3.6 (IO6)
- net ADC_Bat: now reaches U3.7 (IO7)
Other:
- moved on the sheet: C10, C11, C12, C6, C7, C8, C9, J2, R11, R12, R6, R7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

Commit message: routing done?
Connections:
- net AMP_BCLK: now also U3.34 (IO41); no longer U3.33 (IO40)
- net AMP_LRCLK: now also U3.33 (IO40); no longer U3.34 (IO41)
- net EN_A: now also U3.32 (IO39); no longer U3.31 (IO38)
- net EN_B: now also U3.31 (IO38); no longer U3.32 (IO39)
Changed lines of the file:
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@@
-	(wire
-		(pts
-			(xy 95.25 74.93) (xy 96.52 74.93)
-		)
-		(stroke
-			(width 0)
-			(type default)
-		)
-	)
 	(wire
 		(pts
@@
 	(wire
 		(pts
+			(xy 93.98 74.93) (xy 95.25 74.93)
+		)
+		(stroke
+			(width 0)
+			(type default)
+		)
+	)
+	(wire
+		(pts
 			(xy 106.68 88.9) (xy 93.98 88.9)
 		)
@@
 	(wire
 		(pts
-			(xy 93.98 76.2) (xy 95.25 76.2)
-		)
-		(stroke
-			(width 0)
-			(type default)
-		)
-	)
-	(wire
-		(pts
 			(xy 95.25 55.88) (xy 95.25 54.61)
 		)
@@
 	(wire
 		(pts
-			(xy 95.25 76.2) (xy 95.25 74.93)
-		)
-		(stroke
-			(width 0)
-			(type default)
-		)
-	)
-	(wire
-		(pts
 			(xy 95.25 72.39) (xy 101.6 72.39)
 		)
@@
 	(wire
 		(pts
-			(xy 93.98 77.47) (xy 95.25 77.47)
+			(xy 93.98 77.47) (xy 96.52 77.47)
 		)
 		(stroke
@@
 		(pts
 			(xy 40.64 40.64) (xy 40.64 45.72)
+		)
+		(stroke
+			(width 0)
+			(type default)
+		)
+	)
+	(wire
+		(pts
+			(xy 93.98 76.2) (xy 93.98 74.93)
 		)
 		(stroke
@@
 	(hierarchical_label "EN_B"
 		(shape input)
-		(at 101.6 72.39 0)
+		(at 101.6 69.85 0)
 		(effects
 			(font
@@
 	(hierarchical_label "AMP_LRCLK"
 		(shape input)
-		(at 95.25 77.47 0)
+		(at 95.25 74.93 0)
 		(effects
 			(font
@@
 	(hierarchical_label "AMP_BCLK"
 		(shape input)
-		(at 96.52 74.93 0)
+		(at 96.52 77.47 0)
 		(effects
 			(font
@@
 	(hierarchical_label "EN_A"
 		(shape input)
-		(at 101.6 69.85 0)
-		(effects
-			(font
+		(at 101.6 72.39 0)
+		(effects
+			(font

Commit message: more changes!
Connections:
- no-connect marks 6 -> 9
Other:
- note added: "32.768 kHz Crystal"
- note added: "Battery Voltage Sense"
- note added: "Boot Button"
- note added: "Debug Test Points"
- note added: "Display / Touch Connector (FFC2B35-18)"
- note added: "MCU (ESP32-S3-WROOM-1)"
- note added: "Reset Button"
- moved on the sheet: C10, C11, C12, C6, C7, C8, C9, J2, R11, R12, R19, R20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
