File: Anachron/power.kicad_sch (KiCad schematic)
At the start: 22 parts, among them J1 USB4520-03-0-A, Q1 AO3401A, SW1 Pad, U1 AP2112K-3.3TRG1, U2 MCP73831T-2ACI_OT

Commit message: layout power
Parts:
- D1: footprint SOT23-6L_STM -> footprints:SOT23-6L_STM
- J1: footprint USB4520-03-0-A_REVA:GCT_USB4520-03-0-A_REVA -> footprints:GCT_USB4520-03-0-A_REVA
- U1: footprint SOT_RG1_DIO -> footprints:SOT_RG1_DIO
- U2: footprint SOT95P270X145-5N -> footprints:SOT95P270X145-5N
Other:
- moved on the sheet: C4, SW1, U1
