File: Anachron/power.kicad_sch (KiCad schematic)
At the start: 22 parts, among them J1 USB4520-03-0-A, Q1 AO3401A, SW1 Pad, U1 AP2112K-3.3TRG1, U2 MCP73831T-2ACI_OT

Commit message: layout power
Connections:
- net GND: no longer D3.2 (A), Q1.1 (G)
- net VBUS: now also D3.2 (A), Q1.1 (G)
- net C_STAT: now reaches R4.2, U2.1 (STAT)
- net C_PROG: now reaches R3.1, U2.5 (PROG)
Other:
- moved on the sheet: BT1, C3, D2, R4

Commit message: layout power
Parts:
- D2: value LED_Small -> 0603 LED; footprint (none) -> LED_SMD:LED_0603_1608Metric
- R1, R2, R3, R4: footprint Capacitor_SMD:C_0603_1608Metric -> Resistor_SMD:R_0603_1608Metric
Connections:
- net GND: now also R1.2; no longer R1.1
- net CC2: now reaches J1.B5 (CC2)
- net CC2: now also R1.1; no longer R1.2
- net CC1: now reaches J1.A5 (CC1), R2.1
Other:
- note removed: "ADC VOLTAGE DIVIDOR"
- note removed: "FOOTPRINT FOR LED"
- moved on the sheet: C1, R1, R2

Commit message: layed everything outttt
Parts:
- D1: footprint footprints:SOT23-6L_STM -> SOT23-6L_STM
- J1: footprint footprints:GCT_USB4520-03-0-A_REVA -> USB4520-03-0-A_REVA:GCT_USB4520-03-0-A_REVA
- U1: footprint footprints:SOT_RG1_DIO -> SOT_RG1_DIO
- U2: footprint footprints:SOT95P270X145-5N -> SOT95P270X145-5N
Other:
- moved on the sheet: C4, SW1, U1

Commit message: more changes!
Other:
- note added: "3.3V LDO (AP2112K)"
- note added: "Li-ion Charger (MCP73831)"
- note added: "Power Path (VBUS/VBAT to VSYS)"
- note added: "Test Points"
- note added: "USB ESD Protection (USBLC6-2SC6)"
- note added: "USB-C Connector (USB4520)"
- moved on the sheet: BT1, C1, C2, C3, C4, C5, D1, D2, D3, J1, Q1, R1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
