File: Anachron/Anachron.kicad_pcb (KiCad board)
At the start: 4 copper layers, 45 x 47 mm, 18 parts, among them J1 USB4520-03-0-A, Q1 AO3401A, SW1 Pad, U1 AP2112K-3.3TRG1, U2 MCP73831T-2ACI_OT

Commit message: mcu and screen page
Parts:
- added TP1: VBUS, TestPoint:TestPoint_Pad_D1.5mm, F.Cu at (203.6, 134.3)
- added TP2: VBAT, TestPoint:TestPoint_Pad_D1.5mm, F.Cu at (203.6, 137.9)
- added TP3: +3.3V, TestPoint:TestPoint_Pad_D1.5mm, F.Cu at (203.6, 141.4)
Connections:
- net /EN Mode renamed /Power/EN Mode
- net /MCU_D_N renamed /Power/MCU_D_N
- net /MCU_D_P renamed /Power/MCU_D_P
- net /USB_D_N renamed /Power/USB_D_N
- net /USB_D_P renamed /Power/USB_D_P

Commit message: layout power
Parts:
- added C10: 100nF, Capacitor_SMD:C_0805_2012Metric, F.Cu at (243.8, 79.1)
- added C11: 4pF, Capacitor_SMD:C_0805_2012Metric, F.Cu at (134.4, 107.4)
- added C12: 4pF, Capacitor_SMD:C_0805_2012Metric, F.Cu at (132.4, 107.4)
- added C6: 100nF, Capacitor_SMD:C_0603_1608Metric, F.Cu at (126.0, 104.3)
- added C7: 22uF, Capacitor_SMD:C_0805_2012Metric, F.Cu at (127.7, 104.5)
- added C8: 1uF, Capacitor_SMD:C_0603_1608Metric, F.Cu at (243.6, 57.8)
- added C9: 100nF, Capacitor_SMD:C_0805_2012Metric, F.Cu at (243.8, 76.1)
- added J2: FFC2B35-18-G_REVA2, footprints:GCT_FFC2B35-18-G_REVA2, F.Cu at (161.2, 92.0)
- added R10: 0, Capacitor_SMD:C_0603_1608Metric, F.Cu at (130.4, 104.7)
- added R6: 10k, Capacitor_SMD:C_0603_1608Metric, F.Cu at (243.6, 60.3)
- added R7: 10k, Capacitor_SMD:C_0603_1608Metric, F.Cu at (243.6, 62.8)
- added R8: 10k, Capacitor_SMD:C_0603_1608Metric, F.Cu at (243.6, 65.3)
- added R9: 0, Capacitor_SMD:C_0603_1608Metric, F.Cu at (136.4, 104.7)
- added U3: ESP32-S3 N8R8, RF_Module:ESP32-S3-WROOM-1, F.Cu at (128.9, 92.5)
- added Y1: 32.768kHz, footprints:XTAL_SC32S-7PF20PPM_EPS, F.Cu at (133.4, 104.4)
- moved SW1 60.8 mm to (151.2, 104.7), turned to 90 degrees
- moved U1 53.4 mm to (154.8, 104.7)
- moved C4 49.5 mm to (154.8, 102.0)
- moved R5 47.8 mm to (144.7, 104.8), turned to 90 degrees
- moved C5 47.0 mm to (157.8, 104.7), turned to -90 degrees
- moved C2 46.3 mm to (150.8, 109.0), turned to -90 degrees
- moved R3 45.7 mm to (151.5, 111.5), turned to 180 degrees
- moved D3 41.5 mm to (146.5, 107.7), turned to 180 degrees
- moved U2 41.1 mm to (153.8, 109.0), turned to 180 degrees
- moved Q1 40.7 mm to (147.4, 104.3), turned to 90 degrees
- moved BT1 39.2 mm to (199.5, 107.5)
- moved C3 37.9 mm to (200.5, 104.2)
- moved R4 19.6 mm to (198.5, 118.5)
- moved R1 12.5 mm to (134.5, 111.0), turned to 90 degrees
- moved R2 11.6 mm to (136.0, 111.0), turned to -90 degrees
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Connections:
- D3 pad 2: GND -> VBUS
- Q1 pad 1: GND -> VBUS
Other:
- outline, holes or cut-outs redrawn
- board text added: "3V3"
- board text added: "FIND FONT THAT ACC WORKS"

Commit message: layout power
Parts:
- removed R10: 0, Capacitor_SMD:C_0603_1608Metric
- added C13: 100nF, Capacitor_SMD:C_0603_1608Metric, F.Cu at (135.2, 81.8)
- added C14: 100nF, Capacitor_SMD:C_0603_1608Metric, F.Cu at (135.2, 80.2)
- added C15: 100nF, Capacitor_SMD:C_0603_1608Metric, F.Cu at (135.2, 78.8)
- added D2: 0603 LED, LED_SMD:LED_0603_1608Metric, F.Cu at (131.8, 108.5)
- added R11: 100k, Resistor_SMD:R_0603_1608Metric, F.Cu at (152.7, 92.5)
- added R12: 100k, Resistor_SMD:R_0603_1608Metric, F.Cu at (150.5, 93.3)
- added R13: 10k, Resistor_SMD:R_0603_1608Metric, F.Cu at (138.3, 81.8)
- added R14: 10k, Resistor_SMD:R_0603_1608Metric, F.Cu at (138.3, 80.3)
- added R15: 10k, Resistor_SMD:R_0603_1608Metric, F.Cu at (138.3, 78.8)
- added S1: RESET, footprints:SW_TS18-5-25-SL-160-SMT-TR, F.Cu at (149.0, 87.8)
- added S2: BOOT, footprints:SW_TS18-5-25-SL-160-SMT-TR, F.Cu at (149.0, 97.2)
- added S3: Left Button, footprints:PTS845_CNK, F.Cu at (151.6, 74.0)
- added S4: Crown Button, footprints:PTS845_CNK, F.Cu at (143.3, 76.1)
- added S5: Right Button, footprints:PTS845_CNK, F.Cu at (135.1, 74.0)
- BT1: moved to B.Cu
- C10, C11, C12, C9: footprint Capacitor_SMD:C_0805_2012Metric -> Capacitor_SMD:C_0603_1608Metric
- R1, R2, R3, R4, R6, R7, R8, R9: footprint Capacitor_SMD:C_0603_1608Metric -> Resistor_SMD:R_0603_1608Metric
- moved C8 122.8 mm to (129.9, 104.2), turned to 90 degrees
- moved R6 120.5 mm to (131.4, 104.2), turned to 90 degrees
- moved R7 102.7 mm to (145.2, 92.5), turned to 90 degrees
- moved R8 100.1 mm to (147.5, 93.2)
- moved C9 97.6 mm to (147.5, 91.8)
- moved C10 94.2 mm to (150.5, 91.7), turned to 180 degrees
- moved R4 67.7 mm to (131.8, 106.9)
- moved BT1 39.5 mm to (160.2, 102.9), turned to 60 degrees
- moved C3 38.4 mm to (162.1, 102.8), turned to 60 degrees
- moved C12 2.68 mm to (135.1, 107.7)
- moved Y1 2.44 mm to (135.8, 105.0)
- moved C11 2.19 mm to (136.6, 107.7)
- moved U3 1.71 mm to (130.6, 92.5)
- moved R9 1.59 mm to (136.4, 103.1), turned to 180 degrees
- moved C4 0.70 mm to (154.1, 102.0)
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Connections:
- net /MCU + Screen/TP_SCL renamed /MCU + Screen/SCL
- net /MCU + Screen/TP_SDA renamed /MCU + Screen/SDA
- net /MCU + Screen/XTAL_32K_N renamed /MCU + Screen/MCU_OSC_N
- net Net-(C11-Pad1) renamed /MCU + Screen/OSC_N
- net Net-(J1-CC1) renamed /Power/CC1
- net Net-(U2-PROG) renamed /Power/C_PROG
- net Net-(U2-STAT) renamed /Power/C_STAT
- C10 pad 1: /MCU + Screen/BOOT -> /MCU + Screen/Battery ADC
- C12 pad 1: Net-(C12-Pad1) -> /MCU + Screen/MCU_OSC_P
- D1 pad 4: /Power/MCU_D_N -> MCU_D_N
- D1 pad 6: /Power/MCU_D_P -> MCU_D_P
- J1 pad B5: Net-(J1-CC2) -> /Power/CC2
- R1 pad 1: GND -> /Power/CC2
- R1 pad 2: Net-(J1-CC2) -> GND
- U3 pad 13: /MCU + Screen/MCU_D_N -> MCU_D_N
- U3 pad 14: /MCU + Screen/MCU_D_P -> MCU_D_P
- U3 pad 8: /MCU + Screen/XTAL_32K_P -> /MCU + Screen/MCU_OSC_P
- Y1 pad 2: Net-(C12-Pad1) -> /MCU + Screen/MCU_OSC_P
Other:
- outline, holes or cut-outs redrawn
- board text added: "VBUS"
- board text removed: "FIND FONT THAT ACC WORKS"

Commit message: layout power
Parts:
- moved TP2 49.8 mm to (178.8, 94.8)
- moved TP1 49.8 mm to (178.8, 91.2)
- moved TP3 49.8 mm to (178.8, 98.3)
Changed lines of the file:
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@@
 	(footprint "TestPoint:TestPoint_Pad_D1.5mm"
 		(layer "F.Cu")
-		(at 203.6 134.35)
+		(at 178.75 91.25)
 		(descr "SMD pad as test Point, diameter 1.5mm")
 		(tags "test point SMD pad")
@@
 	(footprint "TestPoint:TestPoint_Pad_D1.5mm"
 		(layer "F.Cu")
-		(at 203.6 137.9)
+		(at 178.75 94.8)
 		(descr "SMD pad as test Point, diameter 1.5mm")
 		(tags "test point SMD pad")
@@
 	(footprint "TestPoint:TestPoint_Pad_D1.5mm"
 		(layer "F.Cu")
-		(at 203.6 141.45)
+		(at 178.75 98.35)
 		(descr "SMD pad as test Point, diameter 1.5mm")
 		(tags "test point SMD pad")

Commit message: layed everything outttt
Parts:
- added C16: 100nF, Capacitor_SMD:C_0603_1608Metric, F.Cu at (160.9, 81.5)
- added C17: 10uF, Capacitor_SMD:C_0805_2012Metric, F.Cu at (158.0, 78.5)
- added C20: 100nF, Capacitor_SMD:C_0603_1608Metric, F.Cu at (144.1, 82.0)
- added C21: 100nF, Capacitor_SMD:C_0603_1608Metric, F.Cu at (144.1, 80.5)
- added R16: 22k, Resistor_SMD:R_0603_1608Metric, F.Cu at (135.2, 80.5)
- added R17: 10k, Resistor_SMD:R_0603_1608Metric, F.Cu at (141.2, 82.0)
- added R18: 10k, Resistor_SMD:R_0603_1608Metric, F.Cu at (141.2, 80.5)
- added R19: 10k, Resistor_SMD:R_0603_1608Metric, F.Cu at (129.3, 82.0)
- added R20: 10k, Resistor_SMD:R_0603_1608Metric, F.Cu at (132.2, 82.0)
- added S6: EC05, footprints:EC05 Encoder, B.Cu at (143.3, 73.0)
- added SW2: Pad, Jumper:SolderJumper-2_P1.3mm_Open_RoundedPad1.0x1.5mm, F.Cu at (154.6, 81.6)
- added TP4: TX, TestPoint:TestPoint_Pad_D1.5mm, F.Cu at (185.4, 90.8)
- added TP5: RX, TestPoint:TestPoint_Pad_D1.5mm, F.Cu at (192.2, 90.4)
- added TP6: SDA, TestPoint:TestPoint_Pad_D1.5mm, F.Cu at (185.4, 99.4)
- added TP7: SCL, TestPoint:TestPoint_Pad_D1.5mm, F.Cu at (193.0, 98.6)
- added U4: BMI270, footprints:BMI270_BOS-M, F.Cu at (149.5, 81.5)
- added U5: MAX98357A, Package_DFN_QFN:TQFN-16-1EP_3x3mm_P0.5mm_EP1.23x1.23mm_ThermalVias, F.Cu at (158.0, 81.6)
- R13, R14: value 10k -> 4k7
- moved C15 17.3 mm to (152.4, 81.2), turned to 90 degrees
- moved C14 11.5 mm to (146.7, 81.2), turned to -90 degrees
- moved TP2 6.41 mm to (172.6, 93.0)
- moved C3 4.45 mm to (157.7, 102.1), turned to 180 degrees
- moved C1 4.07 mm to (141.9, 103.8), turned to 0 degrees
- moved TP1 3.45 mm to (178.8, 87.8)
- moved C10 3.33 mm to (153.8, 91.7)
- moved C9 3.33 mm to (150.8, 91.8)
- moved R11 3.33 mm to (156.0, 92.5)
- moved R12 3.33 mm to (153.8, 93.3)
- moved R7 3.33 mm to (148.5, 92.5)
- moved R8 3.33 mm to (150.8, 93.2)
- moved S1 3.33 mm to (152.3, 87.8)
- moved S2 3.33 mm to (152.3, 97.2)
- moved U3 3.33 mm to (133.9, 92.5)
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Connections:
- net MCU_D_N renamed /MCU + Screen/MCU_D_N
- net MCU_D_P renamed /MCU + Screen/MCU_D_P
- C10 pad 1: /MCU + Screen/Battery ADC -> /MCU + Screen/ADC_Bat
- C13 pad 1: /Peripherals/L_Button -> /MCU + Screen/ADC_Button
- C14 pad 1: /Peripherals/C_Button -> +3.3V
- C15 pad 1: /Peripherals/R_Button -> +3.3V
- R11 pad 2: /MCU + Screen/Battery ADC -> /MCU + Screen/ADC_Bat
- R12 pad 1: /MCU + Screen/Battery ADC -> /MCU + Screen/ADC_Bat
- R13 pad 2: /Peripherals/L_Button -> /MCU + Screen/ADC_Button
- R14 pad 1: +3.3V -> /Peripherals/L_Button
- R14 pad 2: /Peripherals/C_Button -> /MCU + Screen/ADC_Button
- R15 pad 1: +3.3V -> /Peripherals/C_Button
- R15 pad 2: /Peripherals/R_Button -> /MCU + Screen/ADC_Button
- U3 pad 10: unconnected-(U3-IO17-Pad10) -> /MCU + Screen/IMU_INT1
- U3 pad 11: unconnected-(U3-IO18-Pad11) -> /MCU + Screen/IMU_INT2
- U3 pad 12: unconnected-(U3-IO8-Pad12) -> /MCU + Screen/AMP_Mode
- U3 pad 17: unconnected-(U3-IO9-Pad17) -> /MCU + Screen/LCD_IO3
- U3 pad 18: unconnected-(U3-IO10-Pad18) -> /MCU + Screen/LCD_CS
- U3 pad 19: unconnected-(U3-IO11-Pad19) -> /MCU + Screen/LCD_IO0
- U3 pad 20: unconnected-(U3-IO12-Pad20) -> /MCU + Screen/LCD_SCLK
- U3 pad 21: unconnected-(U3-IO13-Pad21) -> /MCU + Screen/LCD_IO1
- U3 pad 22: unconnected-(U3-IO14-Pad22) -> /MCU + Screen/LCD_IO2
- U3 pad 23: unconnected-(U3-IO21-Pad23) -> /MCU + Screen/LCD_TE
- U3 pad 24: unconnected-(U3-IO47-Pad24) -> /MCU + Screen/LCD_RST
- U3 pad 25: unconnected-(U3-IO48-Pad25) -> /MCU + Screen/TP_RST
- U3 pad 31: unconnected-(U3-IO38-Pad31) -> /MCU + Screen/EN_A
- U3 pad 32: unconnected-(U3-IO39-Pad32) -> /MCU + Screen/EN_A
- U3 pad 33: unconnected-(U3-IO40-Pad33) -> /MCU + Screen/AMP_BCLK
- U3 pad 34: unconnected-(U3-IO41-Pad34) -> /MCU + Screen/AMP_LRCLK
- U3 pad 35: unconnected-(U3-IO42-Pad35) -> /MCU + Screen/AMP_DIN
- U3 pad 38: unconnected-(U3-IO2-Pad38) -> /MCU + Screen/SDA
- U3 pad 39: unconnected-(U3-IO1-Pad39) -> /MCU + Screen/SCL
- U3 pad 4: unconnected-(U3-IO4-Pad4) -> /MCU + Screen/LCD_BL
- U3 pad 5: unconnected-(U3-IO5-Pad5) -> /MCU + Screen/TP_INT
- U3 pad 6: unconnected-(U3-IO6-Pad6) -> /MCU + Screen/ADC_Button
- U3 pad 7: unconnected-(U3-IO7-Pad7) -> /MCU + Screen/ADC_Bat
Other:
- board text added: "+ -"
- board text added: "- +"
- board text added: "C: 6dB"
- board text added: "NC: 9dB"
- board text added: "SYS PWR"
- board text removed: "3V3"

Commit message: layout power
Parts:
- moved C16 0.55 mm to (161.3, 81.9)
- moved C13 0.38 mm to (134.9, 81.7)
- moved R16 0.38 mm to (134.9, 80.2)
- moved C20 0.38 mm to (143.8, 81.7)
- moved C21 0.38 mm to (143.8, 80.2)
- moved R13 0.38 mm to (137.9, 81.7)
- moved R14 0.38 mm to (137.9, 80.2)
- moved R15 0.38 mm to (137.9, 78.7)
- moved R17 0.38 mm to (140.9, 81.7)
- moved R18 0.38 mm to (140.9, 80.2)
- moved R19 0.38 mm to (129.0, 81.7)
- moved R20 0.38 mm to (132.0, 81.7)
- moved R9 0.28 mm to (138.5, 103.1)
- moved C14 0.25 mm to (146.7, 81.0)
- moved C15 0.25 mm to (152.4, 81.0)
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Routing:
- net VBAT: track 0.00 -> 36.2 mm, vias 0 -> 1
- net /MCU + Screen/LCD_BL: track 0.00 -> 34.7 mm, vias 0 -> 2
- net /MCU + Screen/LCD_SCLK: track 0.00 -> 32.7 mm, vias 0 -> 2
- net /MCU + Screen/LCD_IO0: track 0.00 -> 30.3 mm, vias 0 -> 2
- net /MCU + Screen/LCD_IO2: track 0.00 -> 30.0 mm, vias 0 -> 2
- net /MCU + Screen/LCD_IO1: track 0.00 -> 29.2 mm, vias 0 -> 2
- net +3.3V: track 0.00 -> 29.0 mm, vias 0 -> 2
- net VBUS: track 0.00 -> 22.6 mm, vias 0 -> 6
- net /Power/C_STAT: track 0.00 -> 22.5 mm, vias 0 -> 2
- net /MCU + Screen/LCD_RST: track 0.00 -> 22.2 mm, vias 0 -> 2
- net /MCU + Screen/LCD_CS: track 0.00 -> 19.9 mm, vias 0 -> 2
- net /MCU + Screen/TP_RST: track 0.00 -> 19.6 mm
- net /MCU + Screen/LCD_TE: track 0.00 -> 19.5 mm
- net /Peripherals/L_Button: track 0.00 -> 17.7 mm
- net /MCU + Screen/RESET: track 0.00 -> 13.7 mm
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- added copper zone on F.Cu, net /MCU + Screen/ADC_Button
- added copper zone on In2.Cu, net VBUS
- added copper zone on F.Cu, net VSYS

Commit message: please push
Parts:
- moved C14 4.08 mm to (149.5, 83.9), turned to 0 degrees
Routing:
- net +3.3V: track 29.0 -> 31.2 mm
Changed lines of the file:
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@@
 		(capping no)
 		(filling no)
-		(zone_defaults)
 		(pcbplotparams
 			(layerselection 0x00000000_00000000_55555555_5755f5ff)
@@
 	(footprint "Capacitor_SMD:C_0603_1608Metric"
 		(layer "F.Cu")
-		(at 146.68 80.95 -90)
+		(at 149.5 83.9)
 		(descr "Capacitor SMD 0603 (1608 Metric), square (rectangular) end terminal, IPC-7351 nominal, (Body size source: IPC-SM-782 page 76, https://www.pcb-3d.com/wordpress/wp-content/uploads/ipc-sm-782a_amendment_1_and_2.pdf)")
 		(tags "capacitor")
 		(property "Reference" "C14"
-			(at 0 -1.43 90)
+			(at 0 -1.43 0)
 			(layer "F.SilkS")
 			(hide yes)
@@
 		)
 		(property "Value" "100nF"
-			(at 0 1.43 90)
+			(at 0 1.43 0)
 			(layer "F.Fab")
 			(hide yes)
@@
 		)
 		(property "Datasheet" ""
-			(at 0 0 90)
+			(at 0 0 0)
 			(layer "F.Fab")
 			(hide yes)
@@
 		)
 		(property "Description" "Unpolarized capacitor, small symbol"
-			(at 0 0 90)
+			(at 0 0 0)
 			(layer "F.Fab")
 			(hide yes)
@@
 		)
 		(property "KiLib_Generator" "SMD_2terminal_chip_molded"
-			(at 0 0 90)
+			(at 0 0 0)
 			(layer "F.SilkS")
 			(hide yes)
@@
 		(duplicate_pad_numbers_are_jumpers no)
 		(fp_line
-			(start -0.14058 0.51)
-			(end 0.14058 0.51)
+			(start -0.14058 -0.51)
+			(end 0.14058 -0.51)
 			(stroke
 				(width 0.12)
@@
 		)
 		(fp_line
-			(start -0.14058 -0.51)
-			(end 0.14058 -0.51)
+			(start -0.14058 0.51)
+			(end 0.14058 0.51)
 			(stroke
 				(width 0.12)
@@
 		)
 		(fp_text user "${REFERENCE}"
-			(at 0 0 90)
+			(at 0 0 0)
 			(layer "F.Fab")
 			(effects
@@
 		)
 		(pad "1" smd roundrect
-			(at -0.775 0 270)
+			(at -0.775 0)
 			(size 0.9 0.95)
 			(layers "F.Cu" "F.Mask" "F.Paste")
@@
 		)
 		(pad "2" smd roundrect
-			(at 0.775 0 270)
+			(at 0.775 0)
 			(size 0.9 0.95)
 			(layers "F.Cu" "F.Mask" "F.Paste")
@@
 	)
 	(segment
-		(start 132.4 80.7)
-		(end 132.785 81.085)
+		(start 149.038201 83.586799)
+		(end 148.725 83.9)
 		(width 0.2)
 		(layer "F.Cu")
@@
 	)
 	(segment
-		(start 132.745 103.845)
-		(end 133.25 104.35)
+		(start 132.4 80.7)
+		(end 132.785 81.085)
 		(width 0.2)
 		(layer "F.Cu")
@@
 	)
 	(segment
-		(start 147.054199 80.549199)
-		(end 146.68 80.175)
+		(start 132.745 103.845)
+		(end 133.25 104.35)
 		(width 0.2)
 		(layer "F.Cu")
@@
 	)
 	(segment
+		(start 149.038201 81.761799)
+		(end 149.038201 82.2517)
+		(width 0.2)
+		(layer "F.Cu")
+		(net "+3.3V")
+	)
+	(segment
 		(start 129.96 103.02)
 		(end 130.08 103.14)
@@
 	)
 	(segment
+		(start 150.038199 80.761801)
+		(end 149.038201 81.761799)
+		(width 0.2)
+		(layer "F.Cu")
+		(net "+3.3V")
+	)
+	(segment
 		(start 128.6 80.7)
 		(end 130.48 80.7)
@@
 	)
 	(segment
+		(start 150.038199 80.3467)
+		(end 150.038199 80.761801)
+		(width 0.2)
+		(layer "F.Cu")
+		(net "+3.3V")
+	)
+	(segment
 		(start 159.6475 81.46)
 		(end 160.965 81.46)
@@
 	)
 	(segment
+		(start 149.038201 82.2517)
+		(end 149.038201 83.586799)
+		(width 0.2)
+		(layer "F.Cu")
+		(net "+3.3V")
+	)
+	(segment
 		(start 153.065 81.06)
 		(end 154.81737 81.06)
@@
 		(width 0.2)
 		(layer "F.Cu")
-		(net "+3.3V")
-	)
-	(segment
-		(start 148.3317 80.549199)
-		(end 147.054199 80.549199)
-		(width 0.2)
-		(layer "F.Cu")

Commit message: routing done?
Parts:
- added MP1: Motor Pads, TestPoint:TestPoint_Pad_D2.0mm, B.Cu at (130.6, 92.6)
- TP1, TP2, TP3, TP4, TP5, TP6, TP7: moved to B.Cu
- moved TP5 60.4 mm to (132.4, 82.1), turned to 180 degrees
- moved TP4 49.2 mm to (137.0, 82.1), turned to 180 degrees
- moved TP3 45.4 mm to (133.8, 104.7), turned to 180 degrees
- moved TP1 37.2 mm to (146.0, 105.3), turned to 180 degrees
- moved TP7 36.5 mm to (158.6, 86.4), turned to 180 degrees
- moved TP6 26.6 mm to (162.2, 86.4)
- moved TP2 24.7 mm to (149.5, 101.6), turned to 180 degrees
- moved S1 9.30 mm to (152.3, 97.2)
- moved S2 9.30 mm to (152.3, 87.8), turned to 180 degrees
- moved R7 3.00 mm to (151.5, 92.5), turned to -90 degrees
- moved C9 2.12 mm to (149.3, 93.2), turned to 180 degrees
- moved R8 2.12 mm to (149.3, 91.8), turned to 180 degrees
- moved C17 0.32 mm to (157.6, 78.5)
- moved C1 0.30 mm to (141.9, 103.5)
- moved D1 0.30 mm to (142.0, 106.5)
Connections:
- C20 pad 1: Net-(C20-Pad1) -> /MCU + Screen/EN_B
- R17 pad 2: Net-(C20-Pad1) -> /MCU + Screen/EN_B
- S6 pad B: /MCU + Screen/EN_A -> /MCU + Screen/EN_B
- U3 pad 31: /MCU + Screen/EN_A -> /MCU + Screen/EN_B
- U3 pad 33: /MCU + Screen/AMP_BCLK -> /MCU + Screen/AMP_LRCLK
- U3 pad 34: /MCU + Screen/AMP_LRCLK -> /MCU + Screen/AMP_BCLK
- U5 pad 11: Net-(U5-GND-Pad11) -> GND
- U5 pad 15: Net-(U5-GND-Pad11) -> GND
- U5 pad 8: unconnected-(U5-VDD-Pad8) -> +3.3V
Routing:
- net /MCU + Screen/SCL: track 3.28 -> 53.3 mm, vias 2 -> 3
- net /MCU + Screen/SDA: track 3.37 -> 51.7 mm, vias 2 -> 3
- net /MCU + Screen/TP_INT: track 0.91 -> 44.8 mm, vias 1 -> 2
- net /Peripherals/M-: track 0.00 -> 39.4 mm, vias 0 -> 2
- net /MCU + Screen/ADC_Button: track 0.00 -> 36.3 mm, vias 1 -> 2
- net /Peripherals/M+: track 0.00 -> 35.8 mm, vias 0 -> 2
- net /MCU + Screen/AMP_Mode: track 0.00 -> 33.8 mm, vias 0 -> 2
- net /MCU + Screen/IMU_INT2: track 0.00 -> 28.4 mm, vias 0 -> 2
- net /MCU + Screen/RESET: track 13.7 -> 41.3 mm, vias 0 -> 2
- net /MCU + Screen/AMP_DIN: track 0.00 -> 26.9 mm, vias 0 -> 2
- net /MCU + Screen/IMU_INT1: track 0.00 -> 26.0 mm, vias 0 -> 2
- net /MCU + Screen/ADC_Bat: track 3.04 -> 28.0 mm, vias 0 -> 2
- net /MCU + Screen/AMP_BCLK: track 0.00 -> 24.0 mm, vias 0 -> 2
- net /MCU + Screen/AMP_LRCLK: track 0.00 -> 22.2 mm, vias 0 -> 2
- net /MCU + Screen/EN_B: track 0.00 -> 14.5 mm, vias 0 -> 2
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