File: Anachron/Anachron.kicad_pcb (KiCad board)
At the start: 4 copper layers, 45 x 47 mm, 67 parts, among them J1 USB4520-03-0-A, J2 FFC2B35-18-G_REVA2, Q1 AO3401A, SW1 Pad, SW2 Pad, U1 AP2112K-3.3TRG1, U2 MCP73831T-2ACI_OT, U3 ESP32-S3 N8R8, U4 BMI270, U5 MAX98357A, Y1 32.768kHz

Commit message: pcb pours
Routing:
- net /MCU + Screen/LCD_IO3: track 1.82 -> 35.4 mm, vias 1 -> 2
- net /Power/CC2: track 0.00 -> 14.0 mm, vias 0 -> 2
- net (no net): track 9.60 -> 0.00 mm
- net /Power/CC1: track 0.00 -> 8.32 mm, vias 0 -> 2
- net +3.3V: track 37.1 -> 40.4 mm, vias 3 -> 10
- net /MCU + Screen/BOOT: track 19.4 -> 21.2 mm
- net /Peripherals/M+: track 35.8 -> 37.1 mm
- net /Peripherals/M-: track 39.4 -> 40.2 mm
- net /MCU + Screen/TP_INT: track 44.8 -> 45.5 mm
- net /MCU + Screen/LCD_SCLK: track 32.7 -> 32.0 mm
- net GND: vias 2 -> 3
- added copper zone on In2.Cu, net +3.3V
- added copper zone on B.Cu, net GND
- added copper zone on F.Cu, net GND
- added copper zone on In1.Cu, net GND
